File: TRC2024/Rowpro/ig-normal/PCB_01/ig-normal-ver13_PWM_UARTexpantion.brd (EAGLE design)
At the start: 33 x 67 mm, 37 parts

Commit message: edit
Parts:
- added U1: MAX7315AUET, MAX7315AUET:SOP65P640X110-16N
- moved C3 0.50 mm to (-12.0, 24.0)
- moved R8 0.50 mm to (-11.5, 16.5)
- moved R9 0.40 mm to (-9.90, 24.0)
- moved C5 0.40 mm to (-11.5, 18.6)
- moved C4 0.30 mm to (-11.5, 20.7)
- moved R1 0.30 mm to (-7.80, 24.0)
Connections:
- new net INT: RASPPI.GPIO19, U1.13
- net +3V3: now also U1.16
- net GND: now also U1.1, U1.2, U1.3, U1.8
- net MD1_F: now also U1.4; no longer RASPPI.GPIO5
- net MD1_R: now also U1.5; no longer RASPPI.GPIO6
- net MD2_F: now also U1.6; no longer RASPPI.GPIO25
- net MD2_R: now also U1.7; no longer RASPPI.GPIO16
- net MD3_F: now also U1.9; no longer RASPPI.GPIO17
- net MD3_R: now also U1.10; no longer RASPPI.GPIO27
- net MD4_F: now also U1.11; no longer RASPPI.GPIO23
- net MD4_R: now also U1.12; no longer RASPPI.GPIO24
- net SCL: now also U1.14
- net SDA: now also U1.15
- net SV2: now also RASPPI.GPIO18; no longer RASPPI.GPIO19
Routing:
- net SV2: track 132.6 -> 110.3 mm
- net SDA: track 48.2 -> 68.9 mm, vias 3 -> 6
- net SCL: track 45.8 -> 65.6 mm, vias 3 -> 6
- net MD2_F: track 48.3 -> 29.7 mm
- net +3V3: track 74.8 -> 93.2 mm, vias 2 -> 4
- net INT: track 0.00 -> 15.4 mm
- net GND: track 294.3 -> 307.8 mm, vias 9 -> 10
- net MD3_R: track 32.6 -> 24.4 mm, vias 2 -> 3
- net MD3_F: track 38.0 -> 29.9 mm, vias 2 -> 3
- net MD4_F: track 34.5 -> 26.6 mm, vias 3 -> 4
- net N$7: track 37.6 -> 41.8 mm, vias 3 -> 5
- net MD4_R: track 33.7 -> 30.3 mm, vias 2 -> 4
- net COMV: track 26.2 -> 23.4 mm
- net MD2_R: track 32.3 -> 34.8 mm, vias 2 -> 3
- net +7.4V: track 89.2 -> 91.6 mm, vias 5 -> 4
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- removed copper zone on layer 1, net GND
- removed copper zone on layer 16, net GND
