File: TRC2024/Rowpro/ig-normal/PCB_01/ig-normal-ver13_PWM_UARTexpantion.brd (EAGLE design)
At the start: 33 x 67 mm, 39 parts, among them U1 MAX7315AUET

Commit message: edit brd
Parts:
- removed C5: 470μF-16V, rcl:C0603
- removed R1, R9: 1.2k, rcl:R0805
- added R4, R5: 1.2k, rcl:R0603
- C3: value 10μF-10V -> 10μF
- C4: value 22μF-25v -> 22μF
- R18: value (none) -> BAT
- R19: value (none) -> COM
- R8: value 20k -> 10k
Connections:
- net +5V: now also R4.2; no longer R9.2
- net COMV: no longer C5.1
- net GND: now also R4.1, R5.1; no longer C5.2, R1.1, R9.1
- net TRIM: now also R5.2; no longer R1.2
