File: TRC2024/Rowpro/ig-normal/PCB_01/ig-normal-ver13_PWM_UARTexpantion.sch (EAGLE design)
At the start: 37 parts

Commit message: edit
Parts:
- added U1: MAX7315AUET, MAX7315AUET:MAX7315AUET
Connections:
- new net INT: RASPPI.GPIO19, U1.!INT/08
- net +3V3: now also U1.V+
- net GND: now also U1.AD0, U1.AD1, U1.AD2, U1.GND
- net MD1_F: now also U1.P0; no longer RASPPI.GPIO5
- net MD1_R: now also U1.P1; no longer RASPPI.GPIO6
- net MD2_F: now also U1.P2; no longer RASPPI.GPIO25
- net MD2_R: now also U1.P3; no longer RASPPI.GPIO16
- net MD3_F: now also U1.P4; no longer RASPPI.GPIO17
- net MD3_R: now also U1.P5; no longer RASPPI.GPIO27
- net MD4_F: now also U1.P6; no longer RASPPI.GPIO23
- net MD4_R: now also U1.P7; no longer RASPPI.GPIO24
- net SCL: now also U1.SCL
- net SDA: now also U1.SDA
- net SV2: now also RASPPI.GPIO18; no longer RASPPI.GPIO19
Changed lines of the file:
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@@
 <part name="GND4" library="supply1" library_urn="urn:adsk.eagle:library:371" deviceset="GND" device=""/>
 <part name="CON2" library="con-ml" library_urn="urn:adsk.eagle:library:42302992" deviceset="ML14L" device="" package3d_urn="urn:adsk.eagle:package:42303061/2"/>
+<part name="U1" library="MAX7315AUET" library_urn="urn:adsk.eagle:library:42304147" deviceset="MAX7315AUET" device="" package3d_urn="urn:adsk.eagle:package:42307182/1"/>
+<part name="GND7" library="supply1" library_urn="urn:adsk.eagle:library:371" deviceset="GND" device=""/>
+<part name="+3V7" library="supply1" library_urn="urn:adsk.eagle:library:371" deviceset="+3V3" device=""/>
 </parts>
 <sheets>
@@
 <attribute name="NAME" x="196.85" y="209.042" size="1.778" layer="95"/>
 </instance>
+<instance part="U1" gate="A" x="330.2" y="66.04" smashed="yes">
+<attribute name="NAME" x="317.5" y="87.36" size="2.0828" layer="95" ratio="10" rot="SR0"/>
+<attribute name="VALUE" x="317.5" y="41.72" size="2.0828" layer="96" ratio="10" rot="SR0"/>
+</instance>
+<instance part="GND7" gate="1" x="330.2" y="35.56" smashed="yes">
+<attribute name="VALUE" x="327.66" y="33.02" size="1.778" layer="96"/>
+</instance>
+<instance part="+3V7" gate="G$1" x="350.52" y="88.9" smashed="yes">
+<attribute name="VALUE" x="355.6" y="91.44" size="1.778" layer="96" rot="R180"/>
+</instance>
 </instances>
 <busses>
@@
 <pinref part="GND4" gate="1" pin="GND"/>
 </segment>
+<segment>
+<pinref part="GND7" gate="1" pin="GND"/>
+<wire x1="330.2" y1="38.1" x2="330.2" y2="40.64" width="0.1524" layer="91"/>
+<pinref part="U1" gate="A" pin="AD2"/>
+<wire x1="312.42" y1="73.66" x2="309.88" y2="73.66" width="0.1524" layer="91"/>
+<wire x1="309.88" y1="73.66" x2="309.88" y2="76.2" width="0.1524" layer="91"/>
+<pinref part="U1" gate="A" pin="AD1"/>
+<wire x1="309.88" y1="76.2" x2="312.42" y2="76.2" width="0.1524" layer="91"/>
+<pinref part="U1" gate="A" pin="AD0"/>
+<wire x1="312.42" y1="78.74" x2="309.88" y2="78.74" width="0.1524" layer="91"/>
+<wire x1="309.88" y1="78.74" x2="309.88" y2="76.2" width="0.1524" layer="91"/>
+<junction x="309.88" y="76.2"/>
+<wire x1="309.88" y1="73.66" x2="297.18" y2="73.66" width="0.1524" layer="91"/>
+<wire x1="297.18" y1="73.66" x2="297.18" y2="40.64" width="0.1524" layer="91"/>
+<junction x="309.88" y="73.66"/>
+<wire x1="330.2" y1="40.64" x2="297.18" y2="40.64" width="0.1524" layer="91"/>
+<wire x1="330.2" y1="40.64" x2="350.52" y2="40.64" width="0.1524" layer="91"/>
+<wire x1="350.52" y1="40.64" x2="350.52" y2="50.8" width="0.1524" layer="91"/>
+<pinref part="U1" gate="A" pin="GND"/>
+<wire x1="350.52" y1="50.8" x2="347.98" y2="50.8" width="0.1524" layer="91"/>
+<junction x="330.2" y="40.64"/>
+</segment>
 </net>
 <net name="SDA" class="0">
@@
 <pinref part="ADC" gate="G$1" pin="SCL"/>
 </segment>
+<segment>
+<pinref part="U1" gate="A" pin="SDA"/>
+<wire x1="312.42" y1="53.34" x2="309.88" y2="53.34" width="0.1524" layer="91"/>
+<label x="309.88" y="53.34" size="1.778" layer="95" rot="R180" xref="yes"/>
+</segment>
 </net>
 <net name="SCL" class="0">
@@
 <label x="314.96" y="236.22" size="1.778" layer="95" xref="yes"/>
 <pinref part="ADC" gate="G$1" pin="SDA"/>
+</segment>
+<segment>
+<pinref part="U1" gate="A" pin="SCL"/>
+<wire x1="312.42" y1="71.12" x2="309.88" y2="71.12" width="0.1524" layer="91"/>
+<label x="309.88" y="71.12" size="1.778" layer="95" rot="R180" xref="yes"/>
 </segment>
 </net>
@@
 <wire x1="144.78" y1="162.56" x2="144.78" y2="160.02" width="0.1524" layer="91"/>
 <junction x="144.78" y="160.02"/>
+</segment>
+<segment>
+<pinref part="U1" gate="A" pin="V+"/>
+<wire x1="347.98" y1="83.82" x2="350.52" y2="83.82" width="0.1524" layer="91"/>
+<wire x1="350.52" y1="83.82" x2="350.52" y2="86.36" width="0.1524" layer="91"/>
+<pinref part="+3V7" gate="G$1" pin="+3V3"/>
 </segment>
 </net>
@@
 <net name="MD3_F" class="0">
 <segment>
-<wire x1="27.94" y1="142.24" x2="20.32" y2="142.24" width="0.1524" layer="91"/>
-<label x="20.32" y="142.24" size="1.778" layer="95" rot="R180" xref="yes"/>
-<pinref part="RASPPI" gate="G$1" pin="GPIO17"/>
-</segment>
-<segment>
 <pinref part="MD3" gate="G$1" pin="FIN"/>
 <wire x1="165.1" y1="53.34" x2="152.4" y2="53.34" width="0.1524" layer="91"/>
 <label x="152.4" y="53.34" size="1.4224" layer="95" rot="R180" xref="yes"/>
 </segment>
+<segment>
+<pinref part="U1" gate="A" pin="P4"/>
+<wire x1="347.98" y1="66.04" x2="350.52" y2="66.04" width="0.1524" layer="91"/>
+<label x="350.52" y="66.04" size="1.778" layer="95" xref="yes"/>
+</segment>
 </net>
 <net name="MD1_F" class="0">
@@
 </segment>
 <segment>
-<wire x1="27.94" y1="119.38" x2="22.86" y2="119.38" width="0.1524" layer="91"/>
-<label x="22.86" y="119.38" size="1.778" layer="95" rot="R180" xref="yes"/>
-<pinref part="RASPPI" gate="G$1" pin="GPIO5"/>
+<pinref part="U1" gate="A" pin="P0"/>
+<wire x1="312.42" y1="66.04" x2="309.88" y2="66.04" width="0.1524" layer="91"/>
+<label x="309.88" y="66.04" size="1.778" layer="95" rot="R180" xref="yes"/>
 </segment>
 </net>
@@
 </segment>
 <segment>
-<wire x1="27.94" y1="116.84" x2="22.86" y2="116.84" width="0.1524" layer="91"/>
-<label x="22.86" y="116.84" size="1.778" layer="95" rot="R180" xref="yes"/>
-<pinref part="RASPPI" gate="G$1" pin="GPIO6"/>
+<pinref part="U1" gate="A" pin="P1"/>
+<wire x1="312.42" y1="63.5" x2="309.88" y2="63.5" width="0.1524" layer="91"/>
+<label x="309.88" y="63.5" size="1.778" layer="95" rot="R180" xref="yes"/>
 </segment>
 </net>
@@
 <net name="SV2" class="0">
 <segment>
-<pinref part="RASPPI" gate="G$1" pin="GPIO19"/>
-<wire x1="27.94" y1="111.76" x2="22.86" y2="111.76" width="0.1524" layer="91"/>
-<label x="22.86" y="111.76" size="1.778" layer="95" rot="R180" xref="yes"/>
-</segment>
-<segment>
 <wire x1="208.28" y1="195.58" x2="210.82" y2="195.58" width="0.1524" layer="91"/>
 <label x="210.82" y="195.58" size="1.778" layer="95" xref="yes"/>
 <pinref part="CON2" gate="G$1" pin="5"/>
 <wire x1="208.28" y1="195.58" x2="210.82" y2="195.58" width="0.1524" layer="91"/>
+</segment>
+<segment>
+<pinref part="RASPPI" gate="G$1" pin="GPIO18"/>
+<wire x1="63.5" y1="142.24" x2="68.58" y2="142.24" width="0.1524" layer="91"/>
+<label x="68.58" y="142.24" size="1.778" layer="95" xref="yes"/>
 </segment>
 </net>
@@
 </segment>
 <segment>
-<wire x1="63.5" y1="129.54" x2="68.58" y2="129.54" width="0.1524" layer="91"/>
-<pinref part="RASPPI" gate="G$1" pin="GPIO25"/>
-<label x="68.58" y="129.54" size="1.778" layer="95" xref="yes"/>
+<pinref part="U1" gate="A" pin="P2"/>
+<wire x1="312.42" y1="60.96" x2="309.88" y2="60.96" width="0.1524" layer="91"/>
+<label x="309.88" y="60.96" size="1.778" layer="95" rot="R180" xref="yes"/>
 </segment>
 </net>
@@
 </segment>
 <segment>
-<wire x1="63.5" y1="111.76" x2="68.58" y2="111.76" width="0.1524" layer="91"/>
-<pinref part="RASPPI" gate="G$1" pin="GPIO16"/>
-<label x="68.58" y="111.76" size="1.778" layer="95" xref="yes"/>
+<pinref part="U1" gate="A" pin="P3"/>
+<wire x1="312.42" y1="58.42" x2="309.88" y2="58.42" width="0.1524" layer="91"/>
+<label x="309.88" y="58.42" size="1.778" layer="95" rot="R180" xref="yes"/>
 </segment>
 </net>
 <net name="MD3_R" class="0">
-<segment>
-<wire x1="27.94" y1="139.7" x2="20.32" y2="139.7" width="0.1524" layer="91"/>
-<label x="20.32" y="139.7" size="1.778" layer="95" rot="R180" xref="yes"/>
-<pinref part="RASPPI" gate="G$1" pin="GPIO27"/>
-</segment>
 <segment>
 <pinref part="MD3" gate="G$1" pin="RIN"/>
@@
 <label x="152.4" y="48.26" size="1.4224" layer="95" rot="R180" xref="yes"/>
 </segment>
+<segment>
+<pinref part="U1" gate="A" pin="P5"/>
+<wire x1="347.98" y1="63.5" x2="350.52" y2="63.5" width="0.1524" layer="91"/>
+<label x="350.52" y="63.5" size="1.778" layer="95" xref="yes"/>
+</segment>
 </net>
 <net name="MD4_F" class="0">
@@
 </segment>
 <segment>
-<wire x1="63.5" y1="137.16" x2="68.58" y2="137.16" width="0.1524" layer="91"/>
-<pinref part="RASPPI" gate="G$1" pin="GPIO23"/>
-<label x="68.58" y="137.16" size="1.778" layer="95" xref="yes"/>
+<pinref part="U1" gate="A" pin="P6"/>
+<wire x1="347.98" y1="60.96" x2="350.52" y2="60.96" width="0.1524" layer="91"/>
+<label x="350.52" y="60.96" size="1.778" layer="95" xref="yes"/>
 </segment>
 </net>
@@
 </segment>
 <segment>
-<wire x1="63.5" y1="134.62" x2="68.58" y2="134.62" width="0.1524" layer="91"/>
-<pinref part="RASPPI" gate="G$1" pin="GPIO24"/>
-<label x="68.58" y="134.62" size="1.778" layer="95" xref="yes"/>
+<pinref part="U1" gate="A" pin="P7"/>
+<wire x1="347.98" y1="58.42" x2="350.52" y2="58.42" width="0.1524" layer="91"/>
+<label x="350.52" y="58.42" size="1.778" layer="95" xref="yes"/>
 </segment>
 </net>
@@
 </segment>
 </net>
+<net name="INT" class="0">
+<segment>
+<pinref part="U1" gate="A" pin="!INT/08"/>
+<wire x1="347.98" y1="78.74" x2="350.52" y2="78.74" width="0.1524" layer="91"/>
+<label x="350.52" y="78.74" size="1.778" layer="95" xref="yes"/>
+</segment>
+<segment>
+<pinref part="RASPPI" gate="G$1" pin="GPIO19"/>
+<wire x1="27.94" y1="111.76" x2="22.86" y2="111.76" width="0.1524" layer="91"/>
+<label x="22.86" y="111.76" size="1.778" layer="95" rot="R180" xref="yes"/>
+</segment>
+</net>

Commit message: e
Parts:
- added JP1: (no value), pinhead:PINHD-2X4
Connections:
- net +5V: now also JP1.1
- net CE: now also JP1.6
- net GND: now also JP1.2
- net MISO: now also JP1.4
- net MOSI: now also JP1.3
- net SCL: now also JP1.7
- net SCLK: now also JP1.5
- net SDA: now also JP1.8
Other:
- moved on the sheet: CON1, CON2
