File: TRC2024/Rowpro/ig-normal/PCB_02/ig-normal2ver3.sch (EAGLE design)
At the start: 21 parts

Commit message: l
Parts:
- removed DCDC: OKL-T/6-W12N-CMURATA_OKL-T-6-W12N-C_0_0, OKL-T_6-W12N-C:OKL-T/6-W12N-CMURATA_OKL-T-6-W12N-C_0_0
- added U$1: OKL-T/6-W12N-C_RE, OKL-T_6-W12N-C:OKL-T/6-W12N-C_RE
Connections:
- removed net N$1: BMXCOM.P$1
- removed net N$2: BMXCOM.P$2
- net +3V3: now also BMXCOM.P$4
- net COMV: now also U$1.2_VIN; no longer DCDC.VIN
- net GND: now also U$1.1_ON/OFF, U$1.3_GROUND, U$1.7_GND; no longer DCDC.!ON!/OFF_CONTROL, DCDC.1_GROUND, DCDC.2_GROUND
- net SCL: now also BMXCOM.P$1
- net SDA: now also BMXCOM.P$2
- net TRIM: now also U$1.6_TRIM; no longer DCDC.TRIM
- net VCC: now also U$1.4_VOUT, U$1.5_SENSE; no longer BMXCOM.P$4, DCDC.SENSE, DCDC.VOUT
