File: 13thNSE2024/EAGLE/project/RocketControl/RocketControlver.1(broken).brd (EAGLE design)
At the start: 40 x 50 mm, 16 parts

Commit message: rocketcontroll
Parts:
- added R30, R31: 10k, rcl:R0603
- moved JP2 82.5 mm to (-38.1, -17.8)
- moved LED5 80.3 mm to (-45.7, 40.6)
- moved U$6 71.1 mm to (-35.6, 7.62), turned to 0 degrees
- moved JP1 66.2 mm to (-38.1, -31.8), turned to 0 degrees
- moved R28 61.0 mm to (-26.7, 41.9)
- moved R29 59.7 mm to (-31.8, 41.9)
- moved C17 52.4 mm to (-31.8, 36.8)
- moved C18 49.1 mm to (-44.5, 36.8), turned to 0 degrees
- moved C16 46.4 mm to (-25.4, 36.8), turned to 0 degrees
- moved R26 44.5 mm to (-40.6, 29.2), turned to 0 degrees
- moved R27 43.2 mm to (-21.6, 41.9)
- moved LED6 41.9 mm to (-14.0, 45.7)
- moved PWR2 39.4 mm to (-17.8, 45.7)
- moved U$1 32.1 mm to (-21.6, 16.5)
- moved R25 25.7 mm to (-16.5, 41.9), turned to 0 degrees
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Connections:
- removed net N$6: JP1.8
- net +3V3: now also R30.2, R31.1; no longer JP1.9
- net +5V: no longer JP1.10
- net CANH: no longer JP1.1
- net CANL: no longer JP1.2
- net FP_CHECKER: no longer JP1.5
- net GND: no longer JP1.7
- net PWM: no longer JP1.6
- net SCL2: now also R31.2; no longer JP1.3
- net SDA2: now also R30.1; no longer JP1.4
- net SWDIO2: now also JP2.3; no longer JP2.5
- net SWO2: now also JP2.5; no longer JP2.3
Routing:
- net +3V3: track 110.4 -> 0.00 mm, vias 2 -> 0
- net LED2.1: track 61.4 -> 0.00 mm
- net LED2.0: track 57.1 -> 0.00 mm
- net +5V: track 45.1 -> 0.00 mm
- net FP_CHECKER: track 37.5 -> 0.00 mm
- net SDA2: track 36.6 -> 0.00 mm, vias 1 -> 0
- net SCL2: track 35.0 -> 0.00 mm, vias 1 -> 0
- net PWM: track 30.4 -> 0.00 mm
- net CANL: track 30.0 -> 0.00 mm
- net CANH: track 23.9 -> 0.00 mm
- net TXCAN2: track 22.3 -> 0.00 mm
- net RXCAN2: track 20.7 -> 0.00 mm
- net SWDIO2: track 12.7 -> 0.00 mm
- net SWCLK2: track 11.9 -> 0.00 mm
- net SWO2: track 10.5 -> 0.00 mm
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- removed copper zone on layer 1, net GND
- removed copper zone on layer 16, net GND
Other:
- board text removed: "3v3"
- board text removed: "CLK"
- board text removed: "DIO"
- board text removed: "GND"
- board text removed: "O"
