File: 13thNSE2024/EAGLE/project/RocketControl/RocketControlver.1(broken).sch (EAGLE design)
At the start: 16 parts

Commit message: rocketcontroll
Parts:
- added R30, R31: 10k, rcl:R-US_R0603
Connections:
- removed net N$6: JP1.8
- net +3V3: now also R30.2, R31.1; no longer JP1.9
- net +5V: no longer JP1.10
- net CANH: no longer JP1.1
- net CANL: no longer JP1.2
- net FP_CHECKER: no longer JP1.5
- net GND: no longer JP1.7
- net PWM: no longer JP1.6
- net SCL2: now also R31.2; no longer JP1.3
- net SDA2: now also R30.1; no longer JP1.4
- net SWDIO2: now also JP2.3; no longer JP2.5
- net SWO2: now also JP2.5; no longer JP2.3
